Commit message: fix:

File: src/fire_robot_description/urdf/fire_robot.urdf.xacro (robot description, xacro)
@@ -7,13 +7,17 @@
        - 센서          : RGB 카메라 (Intel RealSense D435 컬러)
                          Depth 카메라 (Intel RealSense D435 뎁스)
-                         Radar (mmWave 2D, 240° FOV, 80m 레인지)
+                         2D LiDAR (/scan, 240° FOV)
        =================================================== -->
-  <xacro:property name="base_length"  value="0.40"/>
-  <xacro:property name="base_width"   value="0.35"/>
-  <xacro:property name="base_height"  value="0.12"/>
-  <xacro:property name="wheel_radius" value="0.07"/>
-  <xacro:property name="wheel_width"  value="0.05"/>
-  <xacro:property name="base_mass"    value="15.0"/>
-  <xacro:property name="wheel_mass"   value="0.5"/>
+  <xacro:property name="base_length"  value="0.420"/>
+  <xacro:property name="base_width"   value="0.310"/>
+  <xacro:property name="base_height"  value="0.184"/>
+  <xacro:property name="wheel_radius" value="0.098"/>
+  <xacro:property name="wheel_width"  value="0.040"/>
+  <xacro:property name="wheelbase"   value="0.262"/>
+  <xacro:property name="track"       value="0.37559"/>
+  <xacro:property name="base_mass"    value="16.523"/>
+  <xacro:property name="wheel_mass"   value="0.477"/>
+  <xacro:property name="camera_z"     value="${base_height/2 + 0.30}"/>
+  <xacro:property name="camera_pitch" value="0.14"/>
   <xacro:macro name="box_inertia" params="m x y z">
     <inertial>
@@ -80,10 +84,10 @@
     </joint>
   </xacro:macro>
-  <xacro:wheel name="front_left"  x_pos="${base_length/2 - 0.05}" y_pos="${base_width/2 + wheel_width/2}"/>
-  <xacro:wheel name="front_right" x_pos="${base_length/2 - 0.05}" y_pos="${-(base_width/2 + wheel_width/2)}"/>
-  <xacro:wheel name="rear_left"   x_pos="${-(base_length/2 - 0.05)}" y_pos="${base_width/2 + wheel_width/2}"/>
-  <xacro:wheel name="rear_right"  x_pos="${-(base_length/2 - 0.05)}" y_pos="${-(base_width/2 + wheel_width/2)}"/>
-  <!-- ============ Radar ============ -->
-  <link name="radar_link">
+  <xacro:wheel name="front_left"  x_pos="${wheelbase/2}" y_pos="${track/2}"/>
+  <xacro:wheel name="front_right" x_pos="${wheelbase/2}" y_pos="${-track/2}"/>
+  <xacro:wheel name="rear_left"   x_pos="${-wheelbase/2}" y_pos="${track/2}"/>
+  <xacro:wheel name="rear_right"  x_pos="${-wheelbase/2}" y_pos="${-track/2}"/>
+  <!-- ============ 2D LiDAR ============ -->
+  <link name="lidar_link">
     <visual>
       <geometry><box size="0.06 0.04 0.02"/></geometry>
@@ -98,8 +102,8 @@
     </inertial>
   </link>
-  <joint name="radar_joint" type="fixed">
+  <joint name="lidar_joint" type="fixed">
     <parent link="base_link"/>
-    <child  link="radar_link"/>
-    <origin xyz="${base_length/2} 0 ${base_height/2 + 0.01}" rpy="0 0 0"/>
+    <child  link="lidar_link"/>
+    <origin xyz="${base_length/2} 0 ${base_height/2 + 0.04}" rpy="0 0 0"/>
   </joint>
   <!-- ============ RGB-D 카메라 마운트 ============ -->
@@ -121,5 +125,5 @@
     <child  link="camera_link"/>
     <!-- 베이스 전방 상단에 전방 하향 8도 틸트 -->
-    <origin xyz="${base_length/2} 0 ${base_height/2 + 0.15}" rpy="0 0.14 0"/>
+    <origin xyz="${base_length/2} 0 ${camera_z}" rpy="0 ${camera_pitch} 0"/>
   </joint>
   <!-- 카메라 광학 프레임 (ROS 컨벤션: Z 앞, X 오른쪽) -->
@@ -128,4 +132,53 @@
     <parent link="camera_link"/>
     <child  link="camera_color_optical_frame"/>
+    <origin xyz="0 0 0" rpy="${-pi/2} 0 ${-pi/2}"/>
+  </joint>
+  <!-- 전방 좌/우 보조 카메라: 벽면 문을 주행 중 미리 보기 위한 45도 시야 -->
+  <link name="camera_front_left_link">
+    <visual>
+      <geometry><box size="0.025 0.080 0.025"/></geometry>
+      <material name="silver"><color rgba="0.8 0.8 0.8 1.0"/></material>
+    </visual>
+    <collision>
+      <geometry><box size="0.025 0.080 0.025"/></geometry>
+    </collision>
+    <inertial>
+      <mass value="0.060"/>
+      <inertia ixx="0.0001" ixy="0" ixz="0" iyy="0.0001" iyz="0" izz="0.0001"/>
+    </inertial>
+  </link>
+  <joint name="camera_front_left_joint" type="fixed">
+    <parent link="base_link"/>
+    <child  link="camera_front_left_link"/>
+    <origin xyz="${base_length/2 - 0.02} 0.20 ${camera_z}" rpy="0 ${camera_pitch} 1.22173"/>
+  </joint>
+  <link name="camera_front_left_optical_frame"/>
+  <joint name="camera_front_left_optical_joint" type="fixed">
+    <parent link="camera_front_left_link"/>
+    <child  link="camera_front_left_optical_frame"/>
+    <origin xyz="0 0 0" rpy="${-pi/2} 0 ${-pi/2}"/>
+  </joint>
+  <link name="camera_front_right_link">
+    <visual>
+      <geometry><box size="0.025 0.080 0.025"/></geometry>
+      <material name="silver"><color rgba="0.8 0.8 0.8 1.0"/></material>
+    </visual>
+    <collision>
+      <geometry><box size="0.025 0.080 0.025"/></geometry>
+    </collision>
+    <inertial>
+      <mass value="0.060"/>
+      <inertia ixx="0.0001" ixy="0" ixz="0" iyy="0.0001" iyz="0" izz="0.0001"/>
+    </inertial>
+  </link>
+  <joint name="camera_front_right_joint" type="fixed">
+    <parent link="base_link"/>
+    <child  link="camera_front_right_link"/>
+    <origin xyz="${base_length/2 - 0.02} -0.20 ${camera_z}" rpy="0 ${camera_pitch} -1.22173"/>
+  </joint>
+  <link name="camera_front_right_optical_frame"/>
+  <joint name="camera_front_right_optical_joint" type="fixed">
+    <parent link="camera_front_right_link"/>
+    <child  link="camera_front_right_optical_frame"/>
     <origin xyz="0 0 0" rpy="${-pi/2} 0 ${-pi/2}"/>
   </joint>
@@ -294,12 +347,12 @@
   </joint>
   <!-- ============ Gazebo Ignition 플러그인 ============ -->
-  <!-- Radar (Ignition gpu_lidar: 240° FOV, 80m, /scan 토픽 → Nav2 호환) -->
-  <gazebo reference="radar_link">
-    <sensor name="radar_sensor" type="gpu_lidar">
+  <!-- 2D LiDAR range sensor (Gazebo uses gpu_lidar internally) -->
+  <gazebo reference="lidar_link">
+    <sensor name="lidar_sensor" type="gpu_lidar">
       <always_on>true</always_on>
       <visualize>false</visualize>
       <update_rate>20</update_rate>
       <topic>scan</topic>
-      <gz_frame_id>radar_link</gz_frame_id>
+      <gz_frame_id>lidar_link</gz_frame_id>
       <lidar>
         <scan>
@@ -319,5 +372,5 @@
         <range>
           <min>0.5</min>
-          <max>80.0</max>
+          <max>12.0</max>
           <resolution>0.05</resolution>
         </range>
@@ -334,5 +387,5 @@
       <always_on>true</always_on>
       <visualize>true</visualize>
-      <update_rate>30</update_rate>
+      <update_rate>15</update_rate>
       <topic>camera_raw</topic>
       <gz_frame_id>camera_color_optical_frame</gz_frame_id>
@@ -340,6 +393,6 @@
         <horizontal_fov>1.204</horizontal_fov>
         <image>
-          <width>640</width>
-          <height>480</height>
+          <width>320</width>
+          <height>240</height>
           <format>R8G8B8</format>
         </image>
@@ -356,4 +409,58 @@
     </sensor>
   </gazebo>
+  <!-- 전방 좌측 카메라 -->
+  <gazebo reference="camera_front_left_link">
+    <sensor name="rgb_camera_front_left" type="camera">
+      <always_on>true</always_on>
+      <visualize>false</visualize>
+      <update_rate>15</update_rate>
+      <topic>camera_front_left_raw</topic>
+      <gz_frame_id>camera_front_left_optical_frame</gz_frame_id>
+      <camera name="rgb_front_left">
+        <horizontal_fov>1.204</horizontal_fov>
+        <image>
+          <width>320</width>
+          <height>240</height>
+          <format>R8G8B8</format>
+        </image>
+        <clip>
+          <near>0.1</near>
+          <far>10.0</far>
+        </clip>
+        <noise>
+          <type>gaussian</type>
+          <mean>0.0</mean>
+          <stddev>0.007</stddev>
+        </noise>
+      </camera>
+    </sensor>
+  </gazebo>
+  <!-- 전방 우측 카메라 -->
+  <gazebo reference="camera_front_right_link">
+    <sensor name="rgb_camera_front_right" type="camera">
+      <always_on>true</always_on>
+      <visualize>false</visualize>
+      <update_rate>15</update_rate>
+      <topic>camera_front_right_raw</topic>
+      <gz_frame_id>camera_front_right_optical_frame</gz_frame_id>
+      <camera name="rgb_front_right">
+        <horizontal_fov>1.204</horizontal_fov>
+        <image>
+          <width>320</width>
+          <height>240</height>
+          <format>R8G8B8</format>
+        </image>
+        <clip>
+          <near>0.1</near>
+          <far>10.0</far>
+        </clip>
+        <noise>
+          <type>gaussian</type>
+          <mean>0.0</mean>
+          <stddev>0.007</stddev>
+        </noise>
+      </camera>
+    </sensor>
+  </gazebo>
   <!-- Depth Camera (Ignition rgbd_camera: RGB + Depth + PointCloud) -->
   <gazebo reference="depth_camera_link">
@@ -361,5 +468,5 @@
       <always_on>true</always_on>
       <visualize>false</visualize>
-      <update_rate>30</update_rate>
+      <update_rate>5</update_rate>
       <topic>depth_camera</topic>
       <gz_frame_id>depth_optical_frame</gz_frame_id>
@@ -367,6 +474,6 @@
         <horizontal_fov>1.204</horizontal_fov>
         <image>
-          <width>640</width>
-          <height>480</height>
+          <width>320</width>
+          <height>240</height>
           <format>R8G8B8</format>
         </image>
@@ -388,8 +495,10 @@
             name="gz::sim::systems::DiffDrive">
       <left_joint>front_left_wheel_joint</left_joint>
+      <left_joint>rear_left_wheel_joint</left_joint>
       <right_joint>front_right_wheel_joint</right_joint>
-      <!-- wheel_separation = 2 × (base_width/2 + wheel_width/2) = 0.40 m -->
-      <wheel_separation>0.40</wheel_separation>
-      <wheel_radius>0.07</wheel_radius>
+      <right_joint>rear_right_wheel_joint</right_joint>
+      <!-- Clearpath j100 reference: track=0.37559 m, wheel_radius=0.098 m -->
+      <wheel_separation>0.37559</wheel_separation>
+      <wheel_radius>0.098</wheel_radius>
       <odom_publish_frequency>20</odom_publish_frequency>
       <topic>cmd_vel</topic>

Commit message: feat: finalize observation-based navigation validation

File: src/fire_robot_description/urdf/fire_robot.urdf.xacro (robot description, xacro)
@@ -20,4 +20,5 @@
   <xacro:property name="camera_z"     value="${base_height/2 + 0.30}"/>
   <xacro:property name="camera_pitch" value="0.14"/>
+  <xacro:property name="enable_sim_depth_camera" value="false"/>
   <xacro:macro name="box_inertia" params="m x y z">
     <inertial>
@@ -352,5 +353,5 @@
       <always_on>true</always_on>
       <visualize>false</visualize>
-      <update_rate>20</update_rate>
+      <update_rate>12</update_rate>
       <topic>scan</topic>
       <gz_frame_id>lidar_link</gz_frame_id>
@@ -371,5 +372,5 @@
         </scan>
         <range>
-          <min>0.5</min>
+          <min>0.15</min>
           <max>12.0</max>
           <resolution>0.05</resolution>
@@ -386,6 +387,6 @@
     <sensor name="rgb_camera" type="camera">
       <always_on>true</always_on>
-      <visualize>true</visualize>
-      <update_rate>15</update_rate>
+      <visualize>false</visualize>
+      <update_rate>6</update_rate>
       <topic>camera_raw</topic>
       <gz_frame_id>camera_color_optical_frame</gz_frame_id>
@@ -414,5 +415,5 @@
       <always_on>true</always_on>
       <visualize>false</visualize>
-      <update_rate>15</update_rate>
+      <update_rate>6</update_rate>
       <topic>camera_front_left_raw</topic>
       <gz_frame_id>camera_front_left_optical_frame</gz_frame_id>
@@ -441,5 +442,5 @@
       <always_on>true</always_on>
       <visualize>false</visualize>
-      <update_rate>15</update_rate>
+      <update_rate>6</update_rate>
       <topic>camera_front_right_raw</topic>
       <gz_frame_id>camera_front_right_optical_frame</gz_frame_id>
@@ -464,4 +465,5 @@
   </gazebo>
   <!-- Depth Camera (Ignition rgbd_camera: RGB + Depth + PointCloud) -->
+  <xacro:if value="${enable_sim_depth_camera}">
   <gazebo reference="depth_camera_link">
     <sensor name="depth_camera" type="rgbd_camera">
@@ -490,4 +492,5 @@
     </sensor>
   </gazebo>
+  </xacro:if>
   <!-- 차동 구동 (Ignition DiffDrive 시스템) -->
   <gazebo>

Commit message: feat: validate observed-handle PIPER door opening

File: src/fire_robot_description/urdf/fire_robot.urdf.xacro (robot description, xacro)
@@ -18,6 +18,6 @@
   <xacro:property name="base_mass"    value="16.523"/>
   <xacro:property name="wheel_mass"   value="0.477"/>
-  <xacro:property name="camera_z"     value="${base_height/2 + 0.30}"/>
-  <xacro:property name="camera_pitch" value="0.14"/>
+  <xacro:property name="camera_z"     value="0.7890"/>
+  <xacro:property name="camera_pitch" value="0.0"/>
   <xacro:property name="enable_sim_depth_camera" value="false"/>
   <xacro:macro name="box_inertia" params="m x y z">
@@ -626,8 +626,6 @@
   </gazebo>
   <!-- Optional sim-only grasp constraint for full door-opening visualization.
-       The physical contact test can publish /fire_robot/sim_arm/handle_attach
-       after the gripper reaches the lever. This is not a pure friction proof;
-       it approximates the gripper maintaining a hold on the lever while the
-       base and arm follow the hinge arc. -->
+       It connects the finger to the articulated lever, not to the door panel,
+       so lever press remains visible while the mobile base supplies the push. -->
   <gazebo>
     <plugin filename="ignition-gazebo-detachable-joint-system"
@@ -635,5 +633,5 @@
       <parent_link>gripper_finger_left</parent_link>
       <child_model>blue_hinged_contact_door</child_model>
-      <child_link>panel</child_link>
+      <child_link>lever</child_link>
       <attach_topic>/fire_robot/sim_arm/handle_attach</attach_topic>
       <detach_topic>/fire_robot/sim_arm/handle_detach</detach_topic>
